File: Front_PD/TR19-PDF_rev1/PDF_rev1.kicad_pcb (KiCad board)
At the start: 2 copper layers, 5 parts, among them J1 Conn_01x11_Female, J2 Conn_01x12_Female

Commit message: PDB FRONT and REAR PCB Layouts
Parts:
- J1: value Conn_01x11_Female -> Conn_01x08_Female; footprint Connector_PinHeader_2.54mm:PinHeader_1x11_P2.54mm_Horizontal -> Connector_PinHeader_2.54mm:PinHeader_1x08_P2.54mm_Horizontal
- J2: value Conn_01x12_Female -> Conn_01x09_Female; footprint Connector_PinHeader_2.54mm:PinHeader_1x12_P2.54mm_Horizontal -> Connector_PinHeader_2.54mm:PinHeader_1x09_P2.54mm_Horizontal
- moved J1 10.9 mm to (99.1, 86.4)
- moved J2 9.67 mm to (160.0, 85.1)
- moved DC1 6.48 mm to (116.4, 106.8)
- moved R1 6.09 mm to (138.0, 110.5)
- moved D1 5.24 mm to (127.0, 110.5)
Routing:
- net Net-(J1-Pad9): track 141.0 -> 0.00 mm
- net Net-(J1-Pad10): track 128.3 -> 0.00 mm
- net Net-(J1-Pad11): track 115.6 -> 0.00 mm
- net Net-(J1-Pad7): track 166.4 -> 120.6 mm
- net Net-(J1-Pad8): track 153.7 -> 107.9 mm
- net Net-(J1-Pad5): track 191.8 -> 146.0 mm
- net Net-(J1-Pad6): track 179.1 -> 133.4 mm
- net Net-(J1-Pad4): track 204.5 -> 158.8 mm
- net Net-(DC1-Pad1): track 158.6 -> 148.5 mm
- net Net-(DC1-Pad7): track 41.6 -> 37.5 mm
- net Net-(J1-Pad1): track 107.9 -> 105.4 mm
- net Net-(D1-Pad2): track 4.26 -> 6.35 mm
- net GND: track 103.6 -> 101.6 mm
Other:
- rule pad_to_mask_clearance: 0.051 -> 0
