File: Front_PD/TR19-PDF_rev1/PDF_rev1.sch (KiCad schematic (older format))
At the start: 5 parts

Commit message: PDB FRONT and REAR PCB Layouts
Parts:
- D1: renamed from D?; footprint (none) -> LED_THT:LED_D3.0mm
- DC1: renamed from DC?; footprint (none) -> TR_Library:445-2487-ND
- J1: renamed from J?; footprint (none) -> Connector_PinHeader_2.54mm:PinHeader_1x08_P2.54mm_Horizontal
- J2: renamed from J?; footprint (none) -> Connector_PinHeader_2.54mm:PinHeader_1x09_P2.54mm_Horizontal
- R1: renamed from R?; footprint (none) -> Resistor_SMD:R_1806_4516Metric_Pad1.57x1.80mm_HandSolder
Changed lines of the file:
@@
 EESchema Schematic File Version 4
+LIBS:PDF_rev1-cache
 EELAYER 26 0
 EELAYER END
@@
 $EndDescr
 $Comp
-L TR-Baja-Components:CC6-1205SR-E DC?
+L TR-Baja-Components:CC6-1205SR-E DC1
 U 1 1 5C570E13
 P 5650 3750
-F 0 "DC?" H 5625 4593 60  0000 C CNN
+F 0 "DC1" H 5625 4593 60  0000 C CNN
 F 1 "CC6-1205SR-E" H 5625 4487 60  0000 C CNN
-F 2 "" H 5550 3750 60  0001 C CNN
+F 2 "TR_Library:445-2487-ND" H 5550 3750 60  0001 C CNN
 F 3 "" H 5650 3850 60  0001 C CNN
 F 4 "5V" H 5625 4381 60  0000 C CNN "Voltage"
@@
 	4800 4150 4450 4150
 $Comp
-L Device:R_US R?
+L Device:R_US R1
 U 1 1 5C570FC5
 P 6950 4650
-F 0 "R?" V 6745 4650 50  0000 C CNN
+F 0 "R1" V 6745 4650 50  0000 C CNN
 F 1 "R_US" V 6836 4650 50  0000 C CNN
-F 2 "" V 6990 4640 50  0001 C CNN
+F 2 "Resistor_SMD:R_1806_4516Metric_Pad1.57x1.80mm_HandSolder" V 6990 4640 50  0001 C CNN
 F 3 "~" H 6950 4650 50  0001 C CNN
 	1    6950 4650
@@
 Connection ~ 6700 4150
 $Comp
-L power:GND #PWR?
+L power:GND #PWR0101
 U 1 1 5C571250
 P 7700 4650
-F 0 "#PWR?" H 7700 4400 50  0001 C CNN
+F 0 "#PWR0101" H 7700 4400 50  0001 C CNN
 F 1 "GND" H 7705 4477 50  0000 C CNN
 F 2 "" H 7700 4650 50  0001 C CNN
@@
 $EndComp
 $Comp
-L Device:LED D?
+L Device:LED D1
 U 1 1 5C5715E1
 P 7400 4650
-F 0 "D?" H 7392 4395 50  0000 C CNN
+F 0 "D1" H 7392 4395 50  0000 C CNN
 F 1 "LED" H 7392 4486 50  0000 C CNN
-F 2 "" H 7400 4650 50  0001 C CNN
+F 2 "LED_THT:LED_D3.0mm" H 7400 4650 50  0001 C CNN
 F 3 "~" H 7400 4650 50  0001 C CNN
 	1    7400 4650
@@
 	4650 3400 4050 3400
 $Comp
-L power:GND #PWR?
+L power:GND #PWR0102
 U 1 1 5C57107A
 P 5600 4650
-F 0 "#PWR?" H 5600 4400 50  0001 C CNN
+F 0 "#PWR0102" H 5600 4400 50  0001 C CNN
 F 1 "GND" H 5605 4477 50  0000 C CNN
 F 2 "" H 5600 4650 50  0001 C CNN
@@
 	5600 4650 4650 4650
 $Comp
-L Connector:Conn_01x09_Female J?
+L Connector:Conn_01x09_Female J2
 U 1 1 5C571501
 P 9100 3800
-F 0 "J?" H 9127 3826 50  0000 L CNN
+F 0 "J2" H 9127 3826 50  0000 L CNN
 F 1 "Conn_01x09_Female" H 9127 3735 50  0000 L CNN
-F 2 "" H 9100 3800 50  0001 C CNN
+F 2 "Connector_PinHeader_2.54mm:PinHeader_1x09_P2.54mm_Horizontal" H 9100 3800 50  0001 C CNN
 F 3 "~" H 9100 3800 50  0001 C CNN
 	1    9100 3800
@@
 	4000 3450 4000 2800
 $Comp
-L Connector:Conn_01x08_Female J?
+L Connector:Conn_01x08_Female J1
 U 1 1 5C5758D1
 P 2250 3750
-F 0 "J?" H 2144 4235 50  0000 C CNN
+F 0 "J1" H 2144 4235 50  0000 C CNN
 F 1 "Conn_01x08_Female" H 2144 4144 50  0000 C CNN
-F 2 "" H 2250 3750 50  0001 C CNN
+F 2 "Connector_PinHeader_2.54mm:PinHeader_1x08_P2.54mm_Horizontal" H 2250 3750 50  0001 C CNN
 F 3 "~" H 2250 3750 50  0001 C CNN
 	1    2250 3750

Commit message: PDB PCB Updates
Connections:
- net GND: no longer D1.1 (K), DC1.3 (-Vin), DC1.5 (-Vout), J1.2 (Pin_2), J2.3 (Pin_3)
- new net: DC1.3 (-Vin), J1.2 (Pin_2)
- new net: D1.1 (K), DC1.5 (-Vout), J2.3 (Pin_3)
Changed lines of the file:
@@
 $EndComp
 Wire Wire Line
-	6450 3650 6550 3650
-Wire Wire Line
 	6450 4150 6700 4150
-Wire Wire Line
-	4800 3400 4650 3400
 Wire Wire Line
 	4800 4150 4450 4150
@@
 Connection ~ 6700 4150
 $Comp
-L power:GND #PWR0101
-U 1 1 5C571250
-P 7700 4650
-F 0 "#PWR0101" H 7700 4400 50  0001 C CNN
-F 1 "GND" H 7705 4477 50  0000 C CNN
-F 2 "" H 7700 4650 50  0001 C CNN
-F 3 "" H 7700 4650 50  0001 C CNN
-	1    7700 4650
-	0    -1   -1   0
-$EndComp
-$Comp
 L Device:LED D1
 U 1 1 5C5715E1
@@
 Wire Wire Line
 	7100 4650 7250 4650
-Wire Wire Line
-	7550 4650 7700 4650
 Text GLabel 9100 3700 2    50   Input ~ 0
 5V
 Text GLabel 9100 3600 2    50   Input ~ 0
 GND
-Wire Wire Line
-	6550 3650 6550 4650
-Wire Wire Line
-	6550 4650 5600 4650
-Wire Wire Line
-	4650 4650 4650 3400
-Connection ~ 6550 3650
-Connection ~ 4650 3400
-Wire Wire Line
-	4650 3400 4050 3400
-$Comp
-L power:GND #PWR0102
-U 1 1 5C57107A
-P 5600 4650
-F 0 "#PWR0102" H 5600 4400 50  0001 C CNN
-F 1 "GND" H 5605 4477 50  0000 C CNN
-F 2 "" H 5600 4650 50  0001 C CNN
-F 3 "" H 5600 4650 50  0001 C CNN
-	1    5600 4650
-	1    0    0    -1
-$EndComp
-Connection ~ 5600 4650
-Wire Wire Line
-	5600 4650 4650 4650
 $Comp
 L Connector:Conn_01x09_Female J2
@@
 	8150 3600 8900 3600
 Wire Wire Line
-	6550 3650 8150 3650
-Wire Wire Line
 	8200 4150 8200 3700
 Wire Wire Line
@@
 Text GLabel 9100 4200 2    50   Input ~ 0
 A3
+Wire Wire Line
+	4050 3400 4800 3400
+Wire Wire Line
+	6450 3650 7750 3650
+Wire Wire Line
+	7550 4650 7750 4650
+Wire Wire Line
+	7750 4650 7750 3650
+Connection ~ 7750 3650
+Wire Wire Line
+	7750 3650 8150 3650
 $EndSCHEMATC
