File: Front_PD/TR19-PDF_rev1/PDF_rev2.kicad_pcb (KiCad board)
At the start: 2 copper layers, 5 parts, among them J1 Conn_01x11_Female, J2 Conn_01x12_Female

Commit message: PDB PCB Updates
Parts:
- J1: value Conn_01x11_Female -> Conn_01x08_Female; footprint Connector_PinHeader_2.54mm:PinHeader_1x11_P2.54mm_Horizontal -> Connector_PinHeader_2.54mm:PinHeader_1x08_P2.54mm_Horizontal
- J2: value Conn_01x12_Female -> Conn_01x09_Female; footprint Connector_PinHeader_2.54mm:PinHeader_1x12_P2.54mm_Horizontal -> Connector_PinHeader_2.54mm:PinHeader_1x09_P2.54mm_Horizontal
- moved J2 17.3 mm to (153.7, 90.2)
- moved J1 16.5 mm to (99.1, 92.7)
- moved DC1 11.7 mm to (112.6, 111.8)
- moved D1 10.2 mm to (125.7, 115.6)
- moved R1 10.2 mm to (134.6, 115.6)
Routing:
- net Net-(J1-Pad4): track 204.5 -> 54.6 mm
- net Net-(J1-Pad9): track 141.0 -> 0.00 mm
- net Net-(J1-Pad5): track 191.8 -> 54.6 mm
- net Net-(J1-Pad10): track 128.3 -> 0.00 mm
- net Net-(J1-Pad6): track 179.1 -> 54.6 mm
- net Net-(J1-Pad11): track 115.6 -> 0.00 mm
- net Net-(J1-Pad7): track 166.4 -> 54.6 mm
- net Net-(J1-Pad8): track 153.7 -> 54.6 mm
- net Net-(DC1-Pad1): track 158.6 -> 77.0 mm
- net Net-(J1-Pad1): track 107.9 -> 57.1 mm
- net GND: track 103.6 -> 80.4 mm
- net Net-(DC1-Pad7): track 41.6 -> 31.8 mm
Other:
- rule pad_to_mask_clearance: 0.051 -> 0

Commit message: PDB PCB Updates
Connections:
- D1 pad 1: GND -> Net-(D1-Pad1)
- DC1 pad 3: GND -> Net-(DC1-Pad3)
- DC1 pad 5: GND -> Net-(D1-Pad1)
- J1 pad 2: GND -> Net-(DC1-Pad3)
- J2 pad 3: GND -> Net-(D1-Pad1)
Routing:
- net GND: track 80.4 -> 0.00 mm
- net Net-(D1-Pad1): track 0.00 -> 47.3 mm
- net Net-(DC1-Pad3): track 0.00 -> 15.1 mm
