File: Rear_PD/TR19-PDR_rev1/TR19-PDR_rev1.sch (KiCad schematic (older format))
At the start: 5 parts

Commit message: PDB FRONT and REAR PCB Layouts
Parts:
- D1: renamed from D?; footprint (none) -> LED_THT:LED_D3.0mm
- DC1: renamed from DC?; footprint (none) -> TR_Library:445-2487-ND
- J1: renamed from J?; footprint (none) -> Connector_PinHeader_2.54mm:PinHeader_1x11_P2.54mm_Horizontal
- J2: renamed from J?; footprint (none) -> Connector_PinHeader_2.54mm:PinHeader_1x12_P2.54mm_Horizontal
- R1: renamed from R?; footprint (none) -> Resistor_SMD:R_1806_4516Metric_Pad1.57x1.80mm_HandSolder
Changed lines of the file:
@@
 EESchema Schematic File Version 4
+LIBS:TR19-PDR_rev1-cache
 EELAYER 26 0
 EELAYER END
@@
 $EndDescr
 $Comp
-L TR-Baja-Components:CC6-1205SR-E DC?
+L TR-Baja-Components:CC6-1205SR-E DC1
 U 1 1 5C59FA59
 P 5600 3450
-F 0 "DC?" H 5575 4293 60  0000 C CNN
+F 0 "DC1" H 5575 4293 60  0000 C CNN
 F 1 "CC6-1205SR-E" H 5575 4187 60  0000 C CNN
-F 2 "" H 5500 3450 60  0001 C CNN
+F 2 "TR_Library:445-2487-ND" H 5500 3450 60  0001 C CNN
 F 3 "" H 5600 3550 60  0001 C CNN
 F 4 "5V" H 5575 4081 60  0000 C CNN "Voltage"
@@
 $EndComp
 $Comp
-L Device:R_US R?
+L Device:R_US R1
 U 1 1 5C59FB1B
 P 7000 4250
-F 0 "R?" V 6795 4250 50  0000 C CNN
+F 0 "R1" V 6795 4250 50  0000 C CNN
 F 1 "R_US" V 6886 4250 50  0000 C CNN
-F 2 "" V 7040 4240 50  0001 C CNN
+F 2 "Resistor_SMD:R_1806_4516Metric_Pad1.57x1.80mm_HandSolder" V 7040 4240 50  0001 C CNN
 F 3 "~" H 7000 4250 50  0001 C CNN
 	1    7000 4250
@@
 $EndComp
 $Comp
-L Device:LED D?
+L Device:LED D1
 U 1 1 5C59FBDA
 P 7450 4250
-F 0 "D?" H 7442 3995 50  0000 C CNN
+F 0 "D1" H 7442 3995 50  0000 C CNN
 F 1 "LED" H 7442 4086 50  0000 C CNN
-F 2 "" H 7450 4250 50  0001 C CNN
+F 2 "LED_THT:LED_D3.0mm" H 7450 4250 50  0001 C CNN
 F 3 "~" H 7450 4250 50  0001 C CNN
 	1    7450 4250
@@
 $EndComp
 $Comp
-L power:GND #PWR?
+L power:GND #PWR0101
 U 1 1 5C59FCD4
 P 7750 4250
-F 0 "#PWR?" H 7750 4000 50  0001 C CNN
+F 0 "#PWR0101" H 7750 4000 50  0001 C CNN
 F 1 "GND" H 7755 4077 50  0000 C CNN
 F 2 "" H 7750 4250 50  0001 C CNN
@@
 Connection ~ 6500 3350
 $Comp
-L power:GND #PWR?
+L power:GND #PWR0102
 U 1 1 5C5A01A6
 P 5500 4300
-F 0 "#PWR?" H 5500 4050 50  0001 C CNN
+F 0 "#PWR0102" H 5500 4050 50  0001 C CNN
 F 1 "GND" H 5505 4127 50  0000 C CNN
 F 2 "" H 5500 4300 50  0001 C CNN
@@
 	3700 4650 8350 4650
 $Comp
-L Connector:Conn_01x12_Female J?
+L Connector:Conn_01x12_Female J2
 U 1 1 5C5A2B2E
 P 9200 4100
-F 0 "J?" H 9227 4076 50  0000 L CNN
+F 0 "J2" H 9227 4076 50  0000 L CNN
 F 1 "Conn_01x12_Female" H 9227 3985 50  0000 L CNN
-F 2 "" H 9200 4100 50  0001 C CNN
+F 2 "Connector_PinHeader_2.54mm:PinHeader_1x12_P2.54mm_Horizontal" H 9200 4100 50  0001 C CNN
 F 3 "~" H 9200 4100 50  0001 C CNN
 	1    9200 4100
@@
 	9000 5700 9000 4700
 $Comp
-L Connector:Conn_01x11_Female J?
+L Connector:Conn_01x11_Female J1
 U 1 1 5C5A93DF
 P 2300 4300
-F 0 "J?" H 2194 4985 50  0000 C CNN
+F 0 "J1" H 2194 4985 50  0000 C CNN
 F 1 "Conn_01x11_Female" H 2194 4894 50  0000 C CNN
-F 2 "" H 2300 4300 50  0001 C CNN
+F 2 "Connector_PinHeader_2.54mm:PinHeader_1x11_P2.54mm_Horizontal" H 2300 4300 50  0001 C CNN
 F 3 "~" H 2300 4300 50  0001 C CNN
 	1    2300 4300

Commit message: PDB PCB Updates
Connections:
- net GND: no longer D1.1 (K), DC1.3 (-Vin), DC1.5 (-Vout), J1.2 (Pin_2), J2.3 (Pin_3)
- new net: DC1.3 (-Vin), J1.2 (Pin_2)
- new net: D1.1 (K), DC1.5 (-Vout), J2.3 (Pin_3)
Changed lines of the file:
@@
 	-1   0    0    1
 $EndComp
-$Comp
-L power:GND #PWR0101
-U 1 1 5C59FCD4
-P 7750 4250
-F 0 "#PWR0101" H 7750 4000 50  0001 C CNN
-F 1 "GND" H 7755 4077 50  0000 C CNN
-F 2 "" H 7750 4250 50  0001 C CNN
-F 3 "" H 7750 4250 50  0001 C CNN
-	1    7750 4250
-	0    -1   -1   0
-$EndComp
 Wire Wire Line
 	7150 4250 7300 4250
@@
 Connection ~ 6600 3850
 Wire Wire Line
-	6400 3350 6500 3350
-Wire Wire Line
-	4750 3100 4500 3100
-Wire Wire Line
 	4750 3850 4650 3850
-Wire Wire Line
-	4500 3100 4500 4300
-Wire Wire Line
-	4500 4300 5500 4300
-Wire Wire Line
-	6500 4300 6500 3350
-Connection ~ 4500 3100
-Connection ~ 6500 3350
-$Comp
-L power:GND #PWR0102
-U 1 1 5C5A01A6
-P 5500 4300
-F 0 "#PWR0102" H 5500 4050 50  0001 C CNN
-F 1 "GND" H 5505 4127 50  0000 C CNN
-F 2 "" H 5500 4300 50  0001 C CNN
-F 3 "" H 5500 4300 50  0001 C CNN
-	1    5500 4300
-	1    0    0    -1
-$EndComp
-Connection ~ 5500 4300
-Wire Wire Line
-	5500 4300 6500 4300
 Wire Wire Line
 	4650 3850 4650 2550
 Connection ~ 4650 3850
-Wire Wire Line
-	3700 4650 8350 4650
 $Comp
 L Connector:Conn_01x12_Female J2
@@
 Wire Wire Line
 	8800 3800 9000 3800
-Wire Wire Line
-	6500 3350 8800 3350
 Wire Wire Line
 	8950 3850 8950 3900
@@
 Wire Wire Line
 	2600 3900 2500 3900
-Wire Wire Line
-	2600 3100 4500 3100
 Wire Wire Line
 	2700 3850 2700 4000
@@
 Text GLabel 9200 4700 2    50   Input ~ 0
 A6
+Wire Wire Line
+	6400 3350 7750 3350
+Wire Wire Line
+	3700 4650 8350 4650
+Wire Wire Line
+	2600 3100 4750 3100
+Wire Wire Line
+	7750 4250 7750 3350
+Connection ~ 7750 3350
+Wire Wire Line
+	7750 3350 8800 3350
 $EndSCHEMATC
