File: Battery_PD/TR19-PDB_rev1/TR19-PDB_rev1.sch (KiCad schematic (older format))
At the start: 12 parts

Commit message: PDB PCB Updates
Parts:
- D4, D5: renamed from D?; footprint (none) -> LED_THT:LED_D3.0mm
- DC1: renamed from DC?; footprint (none) -> TR_Library:1776-2753-ND
- J1: renamed from J?; footprint (none) -> Connector_PinHeader_2.54mm:PinHeader_1x02_P2.54mm_Horizontal
- J2: renamed from J?; footprint (none) -> Connector_PinHeader_2.54mm:PinHeader_1x03_P2.54mm_Horizontal
- R1, R2, R3: renamed from R?; footprint (none) -> Resistor_SMD:R_1806_4516Metric_Pad1.57x1.80mm_HandSolder
- gave numbers to parts that had none: 4
Changed lines of the file:
@@
 EESchema Schematic File Version 4
+LIBS:TR19-PDB_rev1-cache
 EELAYER 26 0
 EELAYER END
@@
 $EndDescr
 $Comp
-L Device:D_Zener D?
+L Device:D_Zener D2
 U 1 1 5C5A00C8
 P 7050 2850
-F 0 "D?" H 7050 2634 50  0000 C CNN
+F 0 "D2" H 7050 2634 50  0000 C CNN
 F 1 "D_Zener" H 7050 2725 50  0000 C CNN
 F 2 "" H 7050 2850 50  0001 C CNN
@@
 $EndComp
 $Comp
-L Device:R_US R?
+L Device:R_US R2
 U 1 1 5C5A01D4
 P 7550 2850
-F 0 "R?" V 7345 2850 50  0000 C CNN
+F 0 "R2" V 7345 2850 50  0000 C CNN
 F 1 "R_US" V 7436 2850 50  0000 C CNN
-F 2 "" V 7590 2840 50  0001 C CNN
+F 2 "Resistor_SMD:R_1806_4516Metric_Pad1.57x1.80mm_HandSolder" V 7590 2840 50  0001 C CNN
 F 3 "~" H 7550 2850 50  0001 C CNN
 	1    7550 2850
@@
 $EndComp
 $Comp
-L Device:LED D?
+L Device:LED D4
 U 1 1 5C5A027B
 P 8050 2850
-F 0 "D?" H 8042 2595 50  0000 C CNN
+F 0 "D4" H 8042 2595 50  0000 C CNN
 F 1 "LED" H 8042 2686 50  0000 C CNN
-F 2 "" H 8050 2850 50  0001 C CNN
+F 2 "LED_THT:LED_D3.0mm" H 8050 2850 50  0001 C CNN
 F 3 "~" H 8050 2850 50  0001 C CNN
 	1    8050 2850
@@
 $EndComp
 $Comp
-L power:GND #PWR?
+L power:GND #PWR0101
 U 1 1 5C5A0371
 P 8400 2850
-F 0 "#PWR?" H 8400 2600 50  0001 C CNN
+F 0 "#PWR0101" H 8400 2600 50  0001 C CNN
 F 1 "GND" V 8405 2722 50  0000 R CNN
 F 2 "" H 8400 2850 50  0001 C CNN
@@
 	6650 4000 8500 4000
 $Comp
-L TR-Baja-Components:SUCW61212B-ND DC?
+L TR-Baja-Components:SUCW61212B-ND DC1
 U 1 1 5C5A0672
 P 5850 3600
-F 0 "DC?" H 5825 4315 50  0000 C CNN
+F 0 "DC1" H 5825 4315 50  0000 C CNN
 F 1 "SUCW61212B-ND" H 5825 4224 50  0000 C CNN
-F 2 "" H 5800 3700 50  0001 C CNN
+F 2 "TR_Library:1776-2753-ND" H 5800 3700 50  0001 C CNN
 F 3 "" H 5800 3700 50  0001 C CNN
 	1    5850 3600
@@
 $EndComp
 $Comp
-L Device:D_Zener D?
+L Device:D_Zener D3
 U 1 1 5C5A0817
 P 7150 4350
-F 0 "D?" H 7150 4134 50  0000 C CNN
+F 0 "D3" H 7150 4134 50  0000 C CNN
 F 1 "D_Zener" H 7150 4225 50  0000 C CNN
 F 2 "" H 7150 4350 50  0001 C CNN
@@
 $EndComp
 $Comp
-L Device:R_US R?
+L Device:R_US R3
 U 1 1 5C5A081E
 P 7650 4350
-F 0 "R?" V 7445 4350 50  0000 C CNN
+F 0 "R3" V 7445 4350 50  0000 C CNN
 F 1 "R_US" V 7536 4350 50  0000 C CNN
-F 2 "" V 7690 4340 50  0001 C CNN
+F 2 "Resistor_SMD:R_1806_4516Metric_Pad1.57x1.80mm_HandSolder" V 7690 4340 50  0001 C CNN
 F 3 "~" H 7650 4350 50  0001 C CNN
 	1    7650 4350
@@
 $EndComp
 $Comp
-L Device:LED D?
+L Device:LED D5
 U 1 1 5C5A0825
 P 8150 4350
-F 0 "D?" H 8142 4095 50  0000 C CNN
+F 0 "D5" H 8142 4095 50  0000 C CNN
 F 1 "LED" H 8142 4186 50  0000 C CNN
-F 2 "" H 8150 4350 50  0001 C CNN
+F 2 "LED_THT:LED_D3.0mm" H 8150 4350 50  0001 C CNN
 F 3 "~" H 8150 4350 50  0001 C CNN
 	1    8150 4350
@@
 $EndComp
 $Comp
-L power:GND #PWR?
+L power:GND #PWR0102
 U 1 1 5C5A082C
 P 7000 4350
-F 0 "#PWR?" H 7000 4100 50  0001 C CNN
+F 0 "#PWR0102" H 7000 4100 50  0001 C CNN
 F 1 "GND" V 7005 4222 50  0000 R CNN
 F 2 "" H 7000 4350 50  0001 C CNN
@@
 Connection ~ 6750 3250
 $Comp
-L power:GND #PWR?
+L power:GND #PWR0103
 U 1 1 5C5A0E54
 P 7650 3500
-F 0 "#PWR?" H 7650 3250 50  0001 C CNN
+F 0 "#PWR0103" H 7650 3250 50  0001 C CNN
 F 1 "GND" H 7655 3327 50  0000 C CNN
 F 2 "" H 7650 3500 50  0001 C CNN
@@
 	3350 4000 3700 4000
 $Comp
-L Device:R_US R?
+L Device:R_US R1
 U 1 1 5C5A1585
 P 3850 3550
-F 0 "R?" V 3645 3550 50  0000 C CNN
+F 0 "R1" V 3645 3550 50  0000 C CNN
 F 1 "R_US" V 3736 3550 50  0000 C CNN
-F 2 "" V 3890 3540 50  0001 C CNN
+F 2 "Resistor_SMD:R_1806_4516Metric_Pad1.57x1.80mm_HandSolder" V 3890 3540 50  0001 C CNN
 F 3 "~" H 3850 3550 50  0001 C CNN
 	1    3850 3550
@@
 $EndComp
 $Comp
-L Switch:SW_SPST SW?
+L Switch:SW_SPST SW1
 U 1 1 5C5A21CD
 P 4200 3550
-F 0 "SW?" H 4200 3785 50  0000 C CNN
+F 0 "SW1" H 4200 3785 50  0000 C CNN
 F 1 "SW_SPST" H 4200 3694 50  0000 C CNN
 F 2 "" H 4200 3550 50  0001 C CNN
@@
 $EndComp
 $Comp
-L Device:D_Zener D?
+L Device:D_Zener D1
 U 1 1 5C5A2317
 P 3950 3800
-F 0 "D?" H 3950 4016 50  0000 C CNN
+F 0 "D1" H 3950 4016 50  0000 C CNN
 F 1 "D_Zener" H 3950 3925 50  0000 C CNN
 F 2 "" H 3950 3800 50  0001 C CNN
@@
 	3700 4000 5000 4000
 $Comp
-L Connector:Conn_01x02_Female J?
+L Connector:Conn_01x02_Female J1
 U 1 1 5C5A38E4
 P 2850 3600
-F 0 "J?" H 2744 3785 50  0000 C CNN
+F 0 "J1" H 2744 3785 50  0000 C CNN
 F 1 "Conn_01x02_Female" H 2744 3694 50  0000 C CNN
-F 2 "" H 2850 3600 50  0001 C CNN
+F 2 "Connector_PinHeader_2.54mm:PinHeader_1x02_P2.54mm_Horizontal" H 2850 3600 50  0001 C CNN
 F 3 "~" H 2850 3600 50  0001 C CNN
 	1    2850 3600
@@
 	3350 3700 3050 3700
 $Comp
-L Connector:Conn_01x03_Female J?
+L Connector:Conn_01x03_Female J2
 U 1 1 5C5A463A
 P 9650 3550
-F 0 "J?" H 9677 3576 50  0000 L CNN
+F 0 "J2" H 9677 3576 50  0000 L CNN
 F 1 "Conn_01x03_Female" H 9677 3485 50  0000 L CNN
-F 2 "" H 9650 3550 50  0001 C CNN
+F 2 "Connector_PinHeader_2.54mm:PinHeader_1x03_P2.54mm_Horizontal" H 9650 3550 50  0001 C CNN
 F 3 "~" H 9650 3550 50  0001 C CNN
 	1    9650 3550

Commit message: PDB PCB Traces
Parts:
- removed SW1: SW_SPST, symbol Switch:SW_SPST
- added J3: SW1, Connector_PinHeader_2.54mm:PinHeader_1x01_P2.54mm_Horizontal, symbol Connector:Conn_01x01_Female
- added J4: SW2, Connector_PinHeader_2.54mm:PinHeader_1x01_P2.54mm_Horizontal, symbol Connector:Conn_01x01_Female
- D1, D2, D3: footprint (none) -> Diode_SMD:D_1806_4516Metric_Pad1.57x1.80mm_HandSolder
Connections:
- net GND: no longer D3.1 (K), D4.1 (K), DC1.5 (COM), J2.2 (Pin_2)
- net at D1.1 (K), DC1.2 (RC): now also J4.1 (Pin_1)
- net at R1.1: now also J3.1 (Pin_1)
- new net: D3.1 (K), D4.1 (K), DC1.5 (COM), J2.2 (Pin_2)
Changed lines of the file:
@@
 F 0 "D2" H 7050 2634 50  0000 C CNN
 F 1 "D_Zener" H 7050 2725 50  0000 C CNN
-F 2 "" H 7050 2850 50  0001 C CNN
+F 2 "Diode_SMD:D_1806_4516Metric_Pad1.57x1.80mm_HandSolder" H 7050 2850 50  0001 C CNN
 F 3 "~" H 7050 2850 50  0001 C CNN
 	1    7050 2850
@@
 	-1   0    0    1
 $EndComp
-$Comp
-L power:GND #PWR0101
-U 1 1 5C5A0371
-P 8400 2850
-F 0 "#PWR0101" H 8400 2600 50  0001 C CNN
-F 1 "GND" V 8405 2722 50  0000 R CNN
-F 2 "" H 8400 2850 50  0001 C CNN
-F 3 "" H 8400 2850 50  0001 C CNN
-	1    8400 2850
-	0    -1   -1   0
-$EndComp
 Wire Wire Line
 	7200 2850 7400 2850
@@
 	7700 2850 7900 2850
 Wire Wire Line
-	8200 2850 8400 2850
-Wire Wire Line
 	6650 3250 6750 3250
-Wire Wire Line
-	6650 3500 7650 3500
 Wire Wire Line
 	6650 4000 8500 4000
@@
 F 0 "D3" H 7150 4134 50  0000 C CNN
 F 1 "D_Zener" H 7150 4225 50  0000 C CNN
-F 2 "" H 7150 4350 50  0001 C CNN
+F 2 "Diode_SMD:D_1806_4516Metric_Pad1.57x1.80mm_HandSolder" H 7150 4350 50  0001 C CNN
 F 3 "~" H 7150 4350 50  0001 C CNN
 	1    7150 4350
@@
 	-1   0    0    1
 $EndComp
-$Comp
-L power:GND #PWR0102
-U 1 1 5C5A082C
-P 7000 4350
-F 0 "#PWR0102" H 7000 4100 50  0001 C CNN
-F 1 "GND" V 7005 4222 50  0000 R CNN
-F 2 "" H 7000 4350 50  0001 C CNN
-F 3 "" H 7000 4350 50  0001 C CNN
-	1    7000 4350
-	0    1    1    0
-$EndComp
 Wire Wire Line
 	7300 4350 7500 4350
@@
 	6750 2850 6750 3250
 Connection ~ 6750 3250
-$Comp
-L power:GND #PWR0103
-U 1 1 5C5A0E54
-P 7650 3500
-F 0 "#PWR0103" H 7650 3250 50  0001 C CNN
-F 1 "GND" H 7655 3327 50  0000 C CNN
-F 2 "" H 7650 3500 50  0001 C CNN
-F 3 "" H 7650 3500 50  0001 C CNN
-	1    7650 3500
-	1    0    0    -1
-$EndComp
-Connection ~ 7650 3500
 Wire Wire Line
 	3350 3250 3700 3250
@@
 $EndComp
 $Comp
-L Switch:SW_SPST SW1
-U 1 1 5C5A21CD
-P 4200 3550
-F 0 "SW1" H 4200 3785 50  0000 C CNN
-F 1 "SW_SPST" H 4200 3694 50  0000 C CNN
-F 2 "" H 4200 3550 50  0001 C CNN
-F 3 "" H 4200 3550 50  0001 C CNN
-	1    4200 3550
-	1    0    0    -1
-$EndComp
-$Comp
 L Device:D_Zener D1
 U 1 1 5C5A2317
@@
 F 0 "D1" H 3950 4016 50  0000 C CNN
 F 1 "D_Zener" H 3950 3925 50  0000 C CNN
-F 2 "" H 3950 3800 50  0001 C CNN
+F 2 "Diode_SMD:D_1806_4516Metric_Pad1.57x1.80mm_HandSolder" H 3950 3800 50  0001 C CNN
 F 3 "~" H 3950 3800 50  0001 C CNN
 	1    3950 3800
@@
 Wire Wire Line
 	9450 3500 9450 3550
-Wire Wire Line
-	7650 3500 9450 3500
 Wire Wire Line
 	9450 4000 9450 3650
@@
 Text GLabel 9650 3650 2    50   Input ~ 0
 -12V
+Wire Wire Line
+	8500 2850 8500 3500
+Wire Wire Line
+	8200 2850 8500 2850
+Connection ~ 8500 3500
+Wire Wire Line
+	8500 3500 9450 3500
+Wire Wire Line
+	6650 3500 7000 3500
+Wire Wire Line
+	7000 4350 7000 3500
+Connection ~ 7000 3500
+Wire Wire Line
+	7000 3500 8500 3500
+$Comp
+L Connector:Conn_01x01_Female J3
+U 1 1 5C7257E0
+P 4200 3550
+F 0 "J3" H 4227 3576 50  0000 L CNN
+F 1 "SW1" H 4227 3485 50  0000 L CNN
+F 2 "Connector_PinHeader_2.54mm:PinHeader_1x01_P2.54mm_Horizontal" H 4200 3550 50  0001 C CNN
+F 3 "~" H 4200 3550 50  0001 C CNN
+	1    4200 3550
+	1    0    0    -1
+$EndComp
+$Comp
+L Connector:Conn_01x01_Female J4
+U 1 1 5C7258B9
+P 4400 3350
+F 0 "J4" V 4340 3262 50  0000 R CNN
+F 1 "SW2" V 4249 3262 50  0000 R CNN
+F 2 "Connector_PinHeader_2.54mm:PinHeader_1x01_P2.54mm_Horizontal" H 4400 3350 50  0001 C CNN
+F 3 "~" H 4400 3350 50  0001 C CNN
+	1    4400 3350
+	0    -1   -1   0
+$EndComp
 $EndSCHEMATC
