File: Competition PDB/TR19-COMP-PD_rev1/TR19-COMP-PD_rev1.kicad_pcb (KiCad board)
At the start: 2 copper layers, 118 parts, among them J1 PWR BTN, J10 RGB_LED3, J11 Sen1, J12 Sen2, J13 Sen3, J14 Sen4, J15 BTN1, J16 BTN2, J17 BTN3, J18 BTN4, J19 BTN5, J2 PWR_LED, J20 BTN6, J21 BTN7, J22 BTN8, J23 BTN9, J24 Sen5, J25 Sen6, J26 Sen7, J27 Sen8, J28 BTN10, J29 BTN11, J3 PTT_LED, J30 BTN12, J31 BTN13, J32 BTN14, J33 BTN15, J34 BTN16, J35 LED1, J36 LED2, J37 LED3, J38 LED4, J39 LED5, J4 Servo1, J40 LED6, J41 LED7, J42 LED8, J43 LED9, J44 LED10, J45 LED11, J46 LED12, J47 LED13, J48 LED14, J49 LED15, J5 Servo2, J50 LED16, J6 Servo3, J7 BATT CONN, J8 RGB_LED1, J9 RGB_LED2, U1 SN74AHCT125_N_14, U2 SN74AHCT125_N_14, U3 SN74AHCT125_N_14, U4 SN74AHCT125_N_14

Commit message: Add pull up resistors for LED drivers
Parts:
- added R61: R_US, Resistor_SMD:R_1210_3225Metric_Pad1.42x2.65mm_HandSolder, F.Cu at (203.1, 49.9)
- added R62: R_US, Resistor_SMD:R_1210_3225Metric_Pad1.42x2.65mm_HandSolder, F.Cu at (203.1, 53.1)
- added R63: R_US, Resistor_SMD:R_1210_3225Metric_Pad1.42x2.65mm_HandSolder, F.Cu at (208.1, 49.9)
- added R64: R_US, Resistor_SMD:R_1210_3225Metric_Pad1.42x2.65mm_HandSolder, F.Cu at (203.1, 56.3)
- added R65: R_US, Resistor_SMD:R_1210_3225Metric_Pad1.42x2.65mm_HandSolder, F.Cu at (208.1, 53.1)
- added R66: R_US, Resistor_SMD:R_1210_3225Metric_Pad1.42x2.65mm_HandSolder, F.Cu at (213.0, 49.9)
- added R67: R_US, Resistor_SMD:R_1210_3225Metric_Pad1.42x2.65mm_HandSolder, F.Cu at (203.1, 59.5)
- added R68: R_US, Resistor_SMD:R_1210_3225Metric_Pad1.42x2.65mm_HandSolder, F.Cu at (208.1, 56.3)
- added R69: R_US, Resistor_SMD:R_1210_3225Metric_Pad1.42x2.65mm_HandSolder, F.Cu at (213.0, 53.1)
- added R70: R_US, Resistor_SMD:R_1210_3225Metric_Pad1.42x2.65mm_HandSolder, F.Cu at (218.0, 49.9)
- added R71: R_US, Resistor_SMD:R_1210_3225Metric_Pad1.42x2.65mm_HandSolder, F.Cu at (208.1, 59.5)
- added R72: R_US, Resistor_SMD:R_1210_3225Metric_Pad1.42x2.65mm_HandSolder, F.Cu at (213.0, 56.3)
- added R73: R_US, Resistor_SMD:R_1210_3225Metric_Pad1.42x2.65mm_HandSolder, F.Cu at (218.0, 53.1)
- added R74: R_US, Resistor_SMD:R_1210_3225Metric_Pad1.42x2.65mm_HandSolder, F.Cu at (213.0, 59.5)
- added R75: R_US, Resistor_SMD:R_1210_3225Metric_Pad1.42x2.65mm_HandSolder, F.Cu at (218.0, 56.3)
- added R76: R_US, Resistor_SMD:R_1210_3225Metric_Pad1.42x2.65mm_HandSolder, F.Cu at (231.1, 67.9)
