File: Competition PDB/TR19-COMP-PD_rev2/TR19-COMP-PD_rev1.sch (KiCad schematic (older format))
At the start: 118 parts, among them J1 PWR BTN, J10 RGB_LED3, J11 Sen1, J12 Sen2, J13 Sen3, J14 Sen4, J15 BTN1, J16 BTN2, J17 BTN3, J18 BTN4, J19 BTN5, J2 PWR_LED, J20 BTN6, J21 BTN7, J22 BTN8, J23 BTN9, J24 Sen5, J25 Sen6, J26 Sen7, J27 Sen8, J28 BTN10, J29 BTN11, J3 PTT_LED, J30 BTN12, J31 BTN13, J32 BTN14, J33 BTN15, J34 BTN16, J35 LED1, J36 LED2, J37 LED3, J38 LED4, J39 LED5, J4 Servo1, J40 LED6, J41 LED7, J42 LED8, J43 LED9, J44 LED10, J45 LED11, J46 LED12, J47 LED13, J48 LED14, J49 LED15, J5 Servo2, J50 LED16, J6 Servo3, J7 BATT CONN, J8 RGB_LED1, J9 RGB_LED2, U1 SN74AHCT125_N_14, U2 SN74AHCT125_N_14, U3 SN74AHCT125_N_14, U4 SN74AHCT125_N_14

Commit message: V2
Version 2 Final update
Parts:
- removed D1: 5V_Zener, Diode_SMD:D_0603_1608Metric_Pad1.05x0.95mm_HandSolder, symbol Device:D_Zener
- removed DC1: SUCW61212B-ND, TR_Library:1776-2753-ND, symbol TR-Baja-Components:SUCW61212B-ND
- removed J43: LED9, Connector_PinHeader_2.54mm:PinHeader_1x02_P2.54mm_Vertical, symbol Connector:Conn_01x02_Female
- removed J44: LED10, Connector_PinHeader_2.54mm:PinHeader_1x02_P2.54mm_Vertical, symbol Connector:Conn_01x02_Female
- removed J45: LED11, Connector_PinHeader_2.54mm:PinHeader_1x02_P2.54mm_Vertical, symbol Connector:Conn_01x02_Female
- removed J46: LED12, Connector_PinHeader_2.54mm:PinHeader_1x02_P2.54mm_Vertical, symbol Connector:Conn_01x02_Female
- removed J47: LED13, Connector_PinHeader_2.54mm:PinHeader_1x02_P2.54mm_Vertical, symbol Connector:Conn_01x02_Female
- removed J48: LED14, Connector_PinHeader_2.54mm:PinHeader_1x02_P2.54mm_Vertical, symbol Connector:Conn_01x02_Female
- removed J49: LED15, Connector_PinHeader_2.54mm:PinHeader_1x02_P2.54mm_Vertical, symbol Connector:Conn_01x02_Female
- removed J50: LED16, Connector_PinHeader_2.54mm:PinHeader_1x02_P2.54mm_Vertical, symbol Connector:Conn_01x02_Female
- removed R1: R1, Resistor_SMD:R_1210_3225Metric_Pad1.42x2.65mm_HandSolder, symbol Device:R_US
- removed R53, R54, R55, R56, R57, R58, R59, R60: R_US, Resistor_SMD:R_1210_3225Metric_Pad1.42x2.65mm_HandSolder, symbol Device:R_US
- removed U1, U2, U3, U4: SN74AHCT125_N_14, TR_Library:SN74AHCT125N, symbol TR-Baja-Components:SN74AHCT125_N_14
- AD1: symbol TR-Baja-Components:ArduinoDue -> TR19-COMP-PD_rev1-rescue:ArduinoDue-TR-Baja-Components
- DC2: symbol TR-Baja-Components:CC6-1205SR-E -> TR19-COMP-PD_rev1-rescue:CC6-1205SR-E-TR-Baja-Components
- J1, J15, J16, J17, J18, J19, J2, J20, J21, J22, J23, J28, J29, J3, J30, J31, J32, J33, J34, J35, J36, J37, J38, J39, J40, J41, J42, J7: footprint Connector_PinHeader_2.54mm:PinHeader_1x02_P2.54mm_Vertical -> Pin_Headers:Pin_Header_Straight_1x02_Pitch2.54mm
- J10, J8, J9: footprint Connector_PinHeader_2.54mm:PinHeader_1x04_P2.54mm_Vertical -> Pin_Headers:Pin_Header_Straight_1x04_Pitch2.54mm
- J11, J12, J13, J14, J24, J25, J26, J27, J4, J5, J6: footprint Connector_PinHeader_2.54mm:PinHeader_1x03_P2.54mm_Vertical -> Pin_Headers:Pin_Header_Straight_1x03_Pitch2.54mm
- R10, R11, R12, R13, R14, R15, R16, R17, R18, R19, R2, R20, R21, R22, R23, R24, R25, R26, R27, R28, R29, R3, R30, R31, R32, R33, R34, R35, R36, R37, R38, R39, R4, R40, R41, R42, R43, R44, R45, R46, R47, R48, R49, R5, R50, R51, R52, R6, R7, R8, R9: footprint Resistor_SMD:R_1210_3225Metric_Pad1.42x2.65mm_HandSolder -> Resistors_SMD:R_1206
Connections:
- net labels removed: DIG10, DIG12, DIG14, DIG16, DIG2, DIG4, DIG6, DIG8, LED10(+), LED11(+), LED12(+), LED13(+), LED14(+), LED15(+), LED16(+), LED9(+)
