File: Competition PDB/TR19-COMP-PD_rev2/TR19-COMP-PD_rev2.kicad_pcb (KiCad board)
At the start: 2 copper layers, 95 parts, among them J1 PWR BTN, J10 RGB_LED3, J11 Sen1, J12 Sen2, J13 Sen3, J14 Sen4, J15 BTN1, J16 BTN2, J17 BTN3, J18 BTN4, J19 BTN5, J2 PWR_LED, J20 BTN6, J21 BTN7, J22 BTN8, J23 BTN9, J24 Sen5, J25 Sen6, J26 Sen7, J27 Sen8, J28 BTN10, J29 BTN11, J3 PTT_LED, J30 BTN12, J31 BTN13, J32 BTN14, J33 BTN15, J34 BTN16, J35 LED1, J36 LED2, J37 LED3, J38 LED4, J39 LED5, J4 Servo1, J40 LED6, J41 LED7, J42 LED8, J5 Servo2, J6 Servo3, J7 BATT CONN, J8 RGB_LED1, J9 RGB_LED2

Commit message: V2 Update
Gerbers
Other:
- board outline added: 102.8 x 56.5 mm
- board text added: "TR Baja 19 Due Shield V2"
Changed lines of the file:
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@@
   (general
     (thickness 1.6)
-    (drawings 0)
+    (drawings 12)
     (tracks 417)
     (zones 0)
@@
   )
   (setup
-    (last_trace_width 0.5)
+    (last_trace_width 0.25)
     (user_trace_width 0.25)
     (user_trace_width 0.5)
@@
       (outputformat 1)
       (mirror false)
-      (drillshape 1)
+      (drillshape 0)
       (scaleselection 1)
       (outputdirectory ""))
@@
     )
   )
+  (gr_text "TR Baja 19\nDue Shield V2" (at 114.05 112.2) (layer F.SilkS)
+    (effects (font (size 1 1) (thickness 0.15)))
+  )
+  (gr_line (start 85.4 67) (end 85.4 67.85) (layer Edge.Cuts) (width 0.1))
+  (gr_line (start 186.4 67) (end 85.4 67) (layer Edge.Cuts) (width 0.1))
+  (gr_line (start 186.4 81.4) (end 186.4 67) (layer Edge.Cuts) (width 0.1))
+  (gr_line (start 188.25 83.25) (end 186.4 81.4) (layer Edge.Cuts) (width 0.1))
+  (gr_line (start 188.25 116.4) (end 188.25 83.25) (layer Edge.Cuts) (width 0.1))
+  (gr_line (start 186.25 118.45) (end 188.25 116.4) (layer Edge.Cuts) (width 0.1))
+  (gr_line (start 186.25 123.45) (end 186.25 118.45) (layer Edge.Cuts) (width 0.1))
+  (gr_line (start 98.45 123.45) (end 186.25 123.45) (layer Edge.Cuts) (width 0.1))
+  (gr_line (start 98.45 108.75) (end 98.45 123.45) (layer Edge.Cuts) (width 0.1))
+  (gr_line (start 85.4 108.8) (end 98.45 108.8) (layer Edge.Cuts) (width 0.1))
+  (gr_line (start 85.4 67.85) (end 85.4 108.8) (layer Edge.Cuts) (width 0.1))
   (segment (start 179.217999 112.484002) (end 179.668001 112.034) (width 0.5) (layer F.Cu) (net 1))
   (segment (start 179.217999 114.815918) (end 179.217999 112.484002) (width 0.5) (layer F.Cu) (net 1))
@@
   (segment (start 90.25 75) (end 90.15 75.1) (width 0.5) (layer F.Cu) (net 40) (status 30))
   (segment (start 97.05 75) (end 90.25 75) (width 0.5) (layer F.Cu) (net 40) (status 30))
-  (segment (start 90.134 97.42) (end 93.03 97.42) (width 0.5) (layer F.Cu) (net 50) (status 10))
-  (via (at 97 93.45) (size 0.8) (drill 0.4) (layers F.Cu B.Cu) (net 50))
-  (segment (start 93.03 97.42) (end 97 93.45) (width 0.5) (layer F.Cu) (net 50))
   (segment (start 116.6 77.08) (end 116.58 77.1) (width 1) (layer B.Cu) (net 41) (status 30))
   (segment (start 116.6 74) (end 116.6 77.08) (width 1) (layer B.Cu) (net 41) (status 30))
@@
   (segment (start 166.214998 84.85) (end 167.089987 83.975011) (width 0.25) (layer B.Cu) (net 49))
   (segment (start 160.69 84.85) (end 166.214998 84.85) (width 0.25) (layer B.Cu) (net 49) (status 10))
+  (segment (start 90.134 97.42) (end 93.03 97.42) (width 0.5) (layer F.Cu) (net 50) (status 10))
+  (via (at 97 93.45) (size 0.8) (drill 0.4) (layers F.Cu B.Cu) (net 50))
+  (segment (start 93.03 97.42) (end 97 93.45) (width 0.5) (layer F.Cu) (net 50))
   (segment (start 99.6 75.01) (end 99.59 75) (width 0.5) (layer F.Cu) (net 50) (status 30))
   (segment (start 99.59 90.86) (end 97 93.45) (width 0.5) (layer B.Cu) (net 50))
